File: TVBGone_KiCAD/TV_B_Gone_ML_v1_2.sch (KiCad schematic (older format))
At the start: 21 parts, among them IC1 ATTINY85, P1 BATT, P2 CONN_3X2, Q1 BC640, Q2 BC548, Q3 BC548, Q4 BC548, Q5 BC548, SW1 START, Y1 8MHz

Commit message: New Design PCB - with Mounting Holes
Totally re-done PCB and footprint files
Parts:
- added P3: PCB, dp_devices:dp_devices-DP5031_V1, symbol CONN_01X01
- added P4, P5, P6, P7: PCB, REInnovationFootprint:NPTH_3MM, symbol CONN_01X01
- C1: footprint (none) -> matts_components:C1V7_lg_pad
- C2: footprint (none) -> matts_components:C1_wide_lg_pad
- D1, D4: value IR wide -> IR; footprint (none) -> REInnovationFootprint:LED-5MM_larg_pad
- D2, D3: value IR narr -> IR; footprint (none) -> REInnovationFootprint:LED-5MM_larg_pad
- D5: footprint (none) -> REInnovationFootprint:LED-5MM_larg_pad
- IC1: footprint DIP8 -> REInnovationFootprint:DIP-8__300_ELL; symbol ATTINY85-P -> ATTINY85-P-RESCUE-TV_B_Gone_ML_v1_2
- P1: value BATT -> BATTERY; footprint (none) -> REInnovationFootprint:conn_2_battery
- P2: value CONN_3X2 -> ISP; footprint (none) -> REInnovationFootprint:TH3x2_ISP
- Q1: footprint (none) -> REInnovationFootprint:TO92-ECB_large_pad_BC639
- Q2, Q3, Q4, Q5: footprint (none) -> REInnovationFootprint:TO92-EBC_large_pad
- R1, R2, R3, R4: footprint (none) -> REInnovationFootprint:TH_Resistor_1
- SW1: footprint (none) -> REInnovationFootprint:SW_PUSH_SMALL_lg_pad
- Y1: footprint (none) -> REInnovationFootprint:SIL-3_lg_pad
Connections:
- no-connect marks 0 -> 5
