File: TVBGone_Hardware/TVBGone_KiCAD/TV_B_Gone_ML_v1_2.sch (KiCad schematic (older format))
At the start: 26 parts, among them IC1 ATTINY85, P1 BATTERY, P2 ISP, P3 PCB, P4 PCB, P5 PCB, P6 PCB, P7 PCB, Q1 BC640, Q2 BC548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

Commit message: Updated PCB files
Parts:
- Q1: symbol PNP -> PNP-RESCUE-TV_B_Gone_ML_v1_2
- Q2, Q3, Q4, Q5: symbol NPN -> NPN-RESCUE-TV_B_Gone_ML_v1_2
Changed lines of the file:
@@
 LIBS:contrib
 LIBS:valves
+LIBS:matts_components
 LIBS:TV_B_Gone_ML_v1_2-cache
 EELAYER 25 0
@@
 $EndComp
 $Comp
-L NPN Q5
+L NPN-RESCUE-TV_B_Gone_ML_v1_2 Q5
 U 1 1 4F15968C
 P 8750 3900
@@
 $EndComp
 $Comp
-L NPN Q4
+L NPN-RESCUE-TV_B_Gone_ML_v1_2 Q4
 U 1 1 4F159689
 P 8750 3200
@@
 $EndComp
 $Comp
-L NPN Q3
+L NPN-RESCUE-TV_B_Gone_ML_v1_2 Q3
 U 1 1 4F159684
 P 8750 2500
@@
 $EndComp
 $Comp
-L PNP Q1
+L PNP-RESCUE-TV_B_Gone_ML_v1_2 Q1
 U 1 1 4F1595EF
 P 7400 4100
@@
 $EndComp
 $Comp
-L NPN Q2
+L NPN-RESCUE-TV_B_Gone_ML_v1_2 Q2
 U 1 1 4F15956A
 P 8750 1800
